Commit message: feat: add dedicated folder for end-effectors

File: robots/common/franka_robot.xacro (robot description, xacro)
@@ -1,5 +1,5 @@
 <?xml version='1.0' encoding='utf-8'?>
 <robot xmlns:xacro="http://www.ros.org/wiki/xacro">
-  <xacro:macro name="franka_robot" params="arm_id joint_limits kinematics inertials dynamics parent:='world' xyz:='0 0 0' rpy:='0 0 0' hand:=false gazebo:=false tcp_xyz:='0 0 0.1034' tcp_rpy:='0 0 0' with_sc:='false' ros2_control:=false robot_ip:='' use_fake_hardware:=false fake_sensor_commands:=false">
+  <xacro:macro name="franka_robot" params="arm_id joint_limits kinematics inertials dynamics parent:='world' xyz:='0 0 0' rpy:='0 0 0' ee_id:=none gazebo:=false with_sc:='false' ros2_control:=false robot_ip:='' use_fake_hardware:=false fake_sensor_commands:=false">
     <xacro:include filename="$(find franka_description)/robots/common/utils.xacro" />
     <xacro:include filename="$(find franka_description)/robots/common/franka_arm.xacro" />
@@ -14,16 +14,47 @@
       with_sc="${with_sc}"
     />
-    <xacro:if value="${hand}">
-      <xacro:include filename="$(find franka_description)/robots/common/franka_hand.xacro"/>
+    <xacro:if value="${ee_id == 'franka_hand'}">
+      <xacro:include filename="$(find franka_description)/end_effectors/common/franka_hand.xacro"/>
+      <xacro:include filename="$(find franka_description)/end_effectors/common/utils.xacro" />
+      <xacro:include filename="$(find franka_description)/end_effectors/$(arg ee_id)/$(arg ee_id)_arguments.xacro" />
+      <xacro:if value="${arm_id == 'fp3'}">
+        <xacro:property name="ee_color" value="black" />
+      </xacro:if>
+      <xacro:if value="${arm_id == 'fr3' or arm_id == 'fer'}">
+        <xacro:property name="ee_color" value="white" />
+      </xacro:if>
       <xacro:franka_hand
+        connected_to="$(arg connection)"
         arm_id="${arm_id}"
-        rpy="0 0 ${-pi/4}"
-        tcp_xyz="${tcp_xyz}"
-        tcp_rpy="${tcp_rpy}"
-        connected_to="${arm_id}_link8"
-        safety_distance="0.03"
+        ee_id="${ee_id}_${ee_color}"
+        ee_inertials="${xacro.load_yaml('$(find franka_description)/end_effectors/$(arg ee_id)/inertials.yaml')}"
+        rpy="$(arg rpy)"
+        xyz="$(arg xyz)"
+        tcp_xyz="$(arg tcp_xyz)"
+        tcp_rpy="$(arg tcp_rpy)"
+        safety_distance="$(arg safety_distance)"
         gazebo="${gazebo}"
+        description_pkg="$(arg description_pkg)"
         with_sc="${with_sc}"
-       />
+      />
+    </xacro:if>
+    <xacro:if value="${ee_id != 'none' and ee_id != 'franka_hand'}">
+      <xacro:include filename="$(find franka_description)/end_effectors/common/ee_with_one_link.xacro"/>
+      <xacro:include filename="$(find franka_description)/end_effectors/common/utils.xacro" />
+      <xacro:include filename="$(find franka_description)/end_effectors/$(arg ee_id)/$(arg ee_id)_arguments.xacro" />
+      <xacro:ee_with_one_link
+        connected_to="$(arg connection)"
+        arm_id="${arm_id}"
+        ee_id="${ee_id}"
+        ee_inertials="${xacro.load_yaml('$(find franka_description)/end_effectors/$(arg ee_id)/inertials.yaml')}"
+        rpy="$(arg rpy)"
+        xyz="$(arg xyz)"
+        tcp_xyz="$(arg tcp_xyz)"
+        tcp_rpy="$(arg tcp_rpy)"
+        safety_distance="$(arg safety_distance)"
+        gazebo="${gazebo}"
+        description_pkg="$(arg description_pkg)"
+        with_sc="${with_sc}"
+      />
     </xacro:if>
     <!-- Definition of additional Gazebo tags -->
@@ -66,5 +97,12 @@
          tip="${arm_id}_joint8"
        />
-      <xacro:if value="${hand}">
+      <xacro:if value="${ee_id == franka_hand_white}">
+        <xacro:gazebo-joint joint="${arm_id}_finger_joint1" transmission="hardware_interface/EffortJointInterface" />
+        <xacro:gazebo-joint joint="${arm_id}_finger_joint2" transmission="hardware_interface/EffortJointInterface" />
+        <!-- Friction specific material for Rubber/Rubber contact -->
+        <xacro:gazebo-friction link="${arm_id}_leftfinger" mu="1.13" />
+        <xacro:gazebo-friction link="${arm_id}_rightfinger" mu="1.13" />
+      </xacro:if>
+      <xacro:if value="${ee_id == franka_hand_black}">
         <xacro:gazebo-joint joint="${arm_id}_finger_joint1" transmission="hardware_interface/EffortJointInterface" />
         <xacro:gazebo-joint joint="${arm_id}_finger_joint2" transmission="hardware_interface/EffortJointInterface" />

File: robots/common/utils.xacro (robot description, xacro)
@@ -37,10 +37,10 @@
       <visual name="${prefix}${name}_visual">
         <geometry>
-          <mesh filename="package://${description_pkg}/meshes/${arm_id}/visual/${name}.dae" />
+          <mesh filename="package://${description_pkg}/meshes/robot_arms/${arm_id}/visual/${name}.dae" />
         </geometry>
       </visual>
       <collision name="${prefix}${name}_collision">
         <geometry>
-          <mesh filename="package://franka_description/meshes/${arm_id}/collision/${name}.stl" />
+          <mesh filename="package://franka_description/meshes/robot_arms/${arm_id}/collision/${name}.stl" />
         </geometry>
       </collision>

File: robots/fer/fer.urdf.xacro (robot description, xacro)
@@ -5,9 +5,5 @@
   <xacro:arg name="arm_id" default="fer" />
   <!-- Should an end-effector be mounted at the flange?" -->
-  <xacro:arg name="hand" default="true" />
-  <!-- Positional offset between $(arm_id)_hand -> $(arm_id)_hand_tcp [m]. Only used when hand:=true -->
-  <xacro:arg name="tcp_xyz" default="0 0 0.1034" />
-  <!-- Rotational offset between $(arm_id)_hand -> $(arm_id)_hand_tcp [rad]. Only used when hand:=true -->
-  <xacro:arg name="tcp_rpy" default="0 0 0" />
+  <xacro:arg name="ee_id" default="none" />
   <!-- Is the robot being simulated in gazebo?" -->
   <xacro:arg name="gazebo" default="false" />
@@ -33,7 +29,5 @@
                       kinematics="${xacro.load_yaml('$(find franka_description)/robots/$(arg arm_id)/kinematics.yaml')}"
                       dynamics="${xacro.load_yaml('$(find franka_description)/robots/$(arg arm_id)/dynamics.yaml')}"
-                      hand="$(arg hand)"
-                      tcp_xyz="$(arg tcp_xyz)"
-                      tcp_rpy="$(arg tcp_rpy)"
+                      ee_id="$(arg ee_id)"
                       with_sc="$(arg with_sc)"
                       ros2_control="$(arg ros2_control)"

File: robots/fp3/fp3.urdf.xacro (robot description, xacro)
@@ -5,9 +5,5 @@
   <xacro:arg name="arm_id" default="fp3" />
   <!-- Should an end-effector be mounted at the flange?" -->
-  <xacro:arg name="hand" default="true" />
-  <!-- Positional offset between $(arm_id)_hand -> $(arm_id)_hand_tcp [m]. Only used when hand:=true -->
-  <xacro:arg name="tcp_xyz" default="0 0 0.1034" />
-  <!-- Rotational offset between $(arm_id)_hand -> $(arm_id)_hand_tcp [rad]. Only used when hand:=true -->
-  <xacro:arg name="tcp_rpy" default="0 0 0" />
+  <xacro:arg name="ee_id" default="none" />
   <!-- Should self-collision be enabled? -->
   <xacro:arg name="with_sc" default="false" />
@@ -25,7 +21,5 @@
                       kinematics="${xacro.load_yaml('$(find franka_description)/robots/$(arg arm_id)/kinematics.yaml')}"
                       dynamics="${xacro.load_yaml('$(find franka_description)/robots/$(arg arm_id)/dynamics.yaml')}"
-                      hand="$(arg hand)"
-                      tcp_xyz="$(arg tcp_xyz)"
-                      tcp_rpy="$(arg tcp_rpy)"
+                      ee_id="$(arg ee_id)"
                       with_sc="$(arg with_sc)"
                       ros2_control="$(arg ros2_control)"

File: robots/fr3/fr3.urdf.xacro (robot description, xacro)
@@ -5,9 +5,5 @@
   <xacro:arg name="arm_id" default="fr3" />
   <!-- Should an end-effector be mounted at the flange?" -->
-  <xacro:arg name="hand" default="true" />
-  <!-- Positional offset between $(arm_id)_hand -> $(arm_id)_hand_tcp [m]. Only used when hand:=true -->
-  <xacro:arg name="tcp_xyz" default="0 0 0.1034" />
-  <!-- Rotational offset between $(arm_id)_hand -> $(arm_id)_hand_tcp [rad]. Only used when hand:=true -->
-  <xacro:arg name="tcp_rpy" default="0 0 0" />
+  <xacro:arg name="ee_id" default="none" />
   <!-- Should self-collision be enabled? -->
   <xacro:arg name="with_sc" default="false" />
@@ -25,7 +21,5 @@
                       kinematics="${xacro.load_yaml('$(find franka_description)/robots/$(arg arm_id)/kinematics.yaml')}"
                       dynamics="${xacro.load_yaml('$(find franka_description)/robots/$(arg arm_id)/dynamics.yaml')}"
-                      hand="$(arg hand)"
-                      tcp_xyz="$(arg tcp_xyz)"
-                      tcp_rpy="$(arg tcp_rpy)"
+                      ee_id="$(arg ee_id)"
                       with_sc="$(arg with_sc)"
                       ros2_control="$(arg ros2_control)"

Commit message: feat: end-effector can be deactivated with an argument

File: robots/common/franka_robot.xacro (robot description, xacro)
@@ -1,5 +1,5 @@
 <?xml version='1.0' encoding='utf-8'?>
 <robot xmlns:xacro="http://www.ros.org/wiki/xacro">
-  <xacro:macro name="franka_robot" params="arm_id joint_limits kinematics inertials dynamics parent:='world' xyz:='0 0 0' rpy:='0 0 0' ee_id:=none gazebo:=false with_sc:='false' ros2_control:=false robot_ip:='' use_fake_hardware:=false fake_sensor_commands:=false">
+  <xacro:macro name="franka_robot" params="arm_id joint_limits kinematics inertials dynamics parent:='world' xyz:='0 0 0' rpy:='0 0 0' hand ee_id:=none gazebo:=false with_sc:='false' ros2_control:=false robot_ip:='' use_fake_hardware:=false fake_sensor_commands:=false">
     <xacro:include filename="$(find franka_description)/robots/common/utils.xacro" />
     <xacro:include filename="$(find franka_description)/robots/common/franka_arm.xacro" />
@@ -14,5 +14,5 @@
       with_sc="${with_sc}"
     />
-    <xacro:if value="${ee_id == 'franka_hand'}">
+    <xacro:if value="${hand and ee_id == 'franka_hand'}">
       <xacro:include filename="$(find franka_description)/end_effectors/common/franka_hand.xacro"/>
       <xacro:include filename="$(find franka_description)/end_effectors/common/utils.xacro" />
@@ -39,5 +39,5 @@
       />
     </xacro:if>
-    <xacro:if value="${ee_id != 'none' and ee_id != 'franka_hand'}">
+    <xacro:if value="${hand and ee_id != 'none' and ee_id != 'franka_hand'}">
       <xacro:include filename="$(find franka_description)/end_effectors/common/ee_with_one_link.xacro"/>
       <xacro:include filename="$(find franka_description)/end_effectors/common/utils.xacro" />

File: robots/fer/fer.urdf.xacro (robot description, xacro)
@@ -5,5 +5,7 @@
   <xacro:arg name="arm_id" default="fer" />
   <!-- Should an end-effector be mounted at the flange?" -->
-  <xacro:arg name="ee_id" default="none" />
+  <xacro:arg name="hand" default="true" />
+  <!-- Which end-effector would be mounted at the flange?" -->
+  <xacro:arg name="ee_id" default="franka_hand" />
   <!-- Is the robot being simulated in gazebo?" -->
   <xacro:arg name="gazebo" default="false" />
@@ -29,4 +31,5 @@
                       kinematics="${xacro.load_yaml('$(find franka_description)/robots/$(arg arm_id)/kinematics.yaml')}"
                       dynamics="${xacro.load_yaml('$(find franka_description)/robots/$(arg arm_id)/dynamics.yaml')}"
+                      hand="$(arg hand)"
                       ee_id="$(arg ee_id)"
                       with_sc="$(arg with_sc)"

File: robots/fp3/fp3.urdf.xacro (robot description, xacro)
@@ -5,5 +5,7 @@
   <xacro:arg name="arm_id" default="fp3" />
   <!-- Should an end-effector be mounted at the flange?" -->
-  <xacro:arg name="ee_id" default="none" />
+  <xacro:arg name="hand" default="true" />
+  <!-- Which end-effector would be mounted at the flange?" -->
+  <xacro:arg name="ee_id" default="franka_hand" />
   <!-- Should self-collision be enabled? -->
   <xacro:arg name="with_sc" default="false" />
@@ -21,4 +23,5 @@
                       kinematics="${xacro.load_yaml('$(find franka_description)/robots/$(arg arm_id)/kinematics.yaml')}"
                       dynamics="${xacro.load_yaml('$(find franka_description)/robots/$(arg arm_id)/dynamics.yaml')}"
+                      hand="$(arg hand)"
                       ee_id="$(arg ee_id)"
                       with_sc="$(arg with_sc)"

File: robots/fr3/fr3.urdf.xacro (robot description, xacro)
@@ -5,5 +5,7 @@
   <xacro:arg name="arm_id" default="fr3" />
   <!-- Should an end-effector be mounted at the flange?" -->
-  <xacro:arg name="ee_id" default="none" />
+  <xacro:arg name="hand" default="true" />
+  <!-- Which end-effector would be mounted at the flange?" -->
+  <xacro:arg name="ee_id" default="franka_hand" />
   <!-- Should self-collision be enabled? -->
   <xacro:arg name="with_sc" default="false" />
@@ -21,4 +23,5 @@
                       kinematics="${xacro.load_yaml('$(find franka_description)/robots/$(arg arm_id)/kinematics.yaml')}"
                       dynamics="${xacro.load_yaml('$(find franka_description)/robots/$(arg arm_id)/dynamics.yaml')}"
+                      hand="$(arg hand)"
                       ee_id="$(arg ee_id)"
                       with_sc="$(arg with_sc)"
