Commit message: Add option to omit arm_id prefix for link, visual, joint elements

File: robots/common/franka_arm.xacro (robot description, xacro)
@@ -8,5 +8,7 @@
   <!-- inertials: description of the inertials that comes from a YAML file. Example definition: ${xacro.load_yaml('$(find franka_description)/robots/fr3/inertials.yaml')} -->
   <!-- dynamics: description of the dynamics that comes from a YAML file. Example definition: ${xacro.load_yaml('$(find franka_description)/robots/fr3/dynamics.yaml')} -->
-  <xacro:macro name="franka_arm" params="arm_id description_pkg:='franka_description' connected_to:='base' xyz:='0 0 0' rpy:='0 0 0' gazebo:='false' safety_distance:=0 joint_limits inertials kinematics dynamics with_sc:=false" >
+  <xacro:macro name="franka_arm" params="arm_id no_prefix:=false description_pkg:='franka_description' connected_to:='base' xyz:='0 0 0' rpy:='0 0 0' gazebo:='false' safety_distance:=0 joint_limits inertials kinematics dynamics with_sc:=false" >
+    <!-- Define a property that defaults to 'arm_id' concatenated with an underscore if 'no_prefix' is not set -->
+    <xacro:property name="prefix" value="${'' if no_prefix else arm_id + '_'}" />
     <xacro:if value="${gazebo}">
       <xacro:property name="connected_to" value="" />
@@ -17,66 +19,66 @@
       <joint name="${connected_to}_joint" type="fixed">
         <parent link="${connected_to}"/>
-        <child link="${arm_id}_link0"/>
+        <child link="${prefix}link0"/>
         <origin rpy="${rpy}" xyz="${xyz}"/>
       </joint>
     </xacro:unless>
-    <xacro:link_with_sc name="link0" gazebo="${gazebo}" with_sc="${with_sc}">
+    <xacro:link_with_sc no_prefix="${no_prefix}" name="link0" gazebo="${gazebo}" with_sc="${with_sc}">
       <self_collision_geometries>
         <xacro:collision_capsule xyz="-0.075 0 0.06" direction="x" radius="${0.06+safety_distance}" length="0.03" />
       </self_collision_geometries>
     </xacro:link_with_sc>
-    <xacro:link_with_sc name="link1" gazebo="${gazebo}" with_sc="${with_sc}">
+    <xacro:link_with_sc no_prefix="${no_prefix}" name="link1" gazebo="${gazebo}" with_sc="${with_sc}">
       <self_collision_geometries>
         <xacro:collision_capsule xyz="0 0 -191.5e-3" radius="${0.06+safety_distance}" length="0.283" />
       </self_collision_geometries>
     </xacro:link_with_sc>
-    <joint name="${arm_id}_joint1" type="revolute">
+    <joint name="${prefix}joint1" type="revolute">
       <xacro:franka-kinematics name="joint1" config="${kinematics}" />
-      <parent link="${arm_id}_link0" />
-      <child link="${arm_id}_link1" />
+      <parent link="${prefix}link0" />
+      <child link="${prefix}link1" />
       <axis xyz="0 0 1" />
       <xacro:franka-limits name="joint1" config="${joint_limits}" />
       <xacro:franka-dynamics name="joint1" config="${dynamics}" />
     </joint>
-    <xacro:link_with_sc name="link2" gazebo="${gazebo}" with_sc="${with_sc}">
+    <xacro:link_with_sc no_prefix="${no_prefix}" name="link2" gazebo="${gazebo}" with_sc="${with_sc}">
       <self_collision_geometries>
         <xacro:collision_capsule xyz="0 0 0" radius="${0.06+safety_distance}" length="0.12" />
       </self_collision_geometries>
     </xacro:link_with_sc>
-    <joint name="${arm_id}_joint2" type="revolute">
+    <joint name="${prefix}joint2" type="revolute">
       <xacro:franka-kinematics name="joint2" config="${kinematics}" />
-      <parent link="${arm_id}_link1" />
-      <child link="${arm_id}_link2" />
+      <parent link="${prefix}link1" />
+      <child link="${prefix}link2" />
       <axis xyz="0 0 1" />
       <xacro:franka-limits name="joint2" config="${joint_limits}" />
       <xacro:franka-dynamics name="joint2" config="${dynamics}" />
     </joint>
-    <xacro:link_with_sc name="link3" gazebo="${gazebo}" with_sc="${with_sc}">
+    <xacro:link_with_sc no_prefix="${no_prefix}" name="link3" gazebo="${gazebo}" with_sc="${with_sc}">
       <self_collision_geometries>
         <xacro:collision_capsule xyz="0 0 -0.145" radius="${0.06+safety_distance}" length="0.15" />
       </self_collision_geometries>
     </xacro:link_with_sc>
-    <joint name="${arm_id}_joint3" type="revolute">
+    <joint name="${prefix}joint3" type="revolute">
       <xacro:franka-kinematics name="joint3" config="${kinematics}" />
-      <parent link="${arm_id}_link2" />
-      <child link="${arm_id}_link3" />
+      <parent link="${prefix}link2" />
+      <child link="${prefix}link3" />
       <axis xyz="0 0 1" />
       <xacro:franka-limits name="joint3" config="${joint_limits}" />
       <xacro:franka-dynamics name="joint3" config="${dynamics}" />
     </joint>
-    <xacro:link_with_sc name="link4" gazebo="${gazebo}" with_sc="${with_sc}">
+    <xacro:link_with_sc no_prefix="${no_prefix}" name="link4" gazebo="${gazebo}" with_sc="${with_sc}">
       <self_collision_geometries>
         <xacro:collision_capsule xyz="0 0 0" radius="${0.06+safety_distance}" length="0.12" />
      </self_collision_geometries>
     </xacro:link_with_sc>
-    <joint name="${arm_id}_joint4" type="revolute">
+    <joint name="${prefix}joint4" type="revolute">
       <xacro:franka-kinematics name="joint4" config="${kinematics}" />
-      <parent link="${arm_id}_link3" />
-      <child link="${arm_id}_link4" />
+      <parent link="${prefix}link3" />
+      <child link="${prefix}link4" />
       <axis xyz="0 0 1" />
       <xacro:franka-limits name="joint4" config="${joint_limits}" />
       <xacro:franka-dynamics name="joint4" config="${dynamics}" />
     </joint>
-    <xacro:link_with_sc name="link5" gazebo="${gazebo}" with_sc="${with_sc}">
+    <xacro:link_with_sc no_prefix="${no_prefix}" name="link5" gazebo="${gazebo}" with_sc="${with_sc}">
       <self_collision_geometries>
         <xacro:collision_capsule xyz="0 0 -0.26"    radius="${0.060+safety_distance}" length="0.10" />
@@ -84,26 +86,26 @@
       </self_collision_geometries>
     </xacro:link_with_sc>
-    <joint name="${arm_id}_joint5" type="revolute">
+    <joint name="${prefix}joint5" type="revolute">
       <xacro:franka-kinematics name="joint5" config="${kinematics}" />
-      <parent link="${arm_id}_link4" />
-      <child link="${arm_id}_link5" />
+      <parent link="${prefix}link4" />
+      <child link="${prefix}link5" />
       <axis xyz="0 0 1" />
       <xacro:franka-limits name="joint5" config="${joint_limits}" />
       <xacro:franka-dynamics name="joint5" config="${dynamics}" />
     </joint>
-    <xacro:link_with_sc name="link6" gazebo="${gazebo}" with_sc="${with_sc}">
+    <xacro:link_with_sc no_prefix="${no_prefix}" name="link6" gazebo="${gazebo}" with_sc="${with_sc}">
       <self_collision_geometries>
         <xacro:collision_capsule xyz="0 0 -0.03" radius="${0.05+safety_distance}" length="0.08" />
       </self_collision_geometries>
     </xacro:link_with_sc>
-    <joint name="${arm_id}_joint6" type="revolute">
+    <joint name="${prefix}joint6" type="revolute">
       <xacro:franka-kinematics name="joint6" config="${kinematics}" />
-      <parent link="${arm_id}_link5" />
-      <child link="${arm_id}_link6" />
+      <parent link="${prefix}link5" />
+      <child link="${prefix}link6" />
       <axis xyz="0 0 1" />
       <xacro:franka-limits name="joint6" config="${joint_limits}" />
       <xacro:franka-dynamics name="joint6" config="${dynamics}" />
     </joint>
-    <xacro:link_with_sc name="link7" gazebo="${gazebo}" rpy="0 0 ${pi/4}" with_sc="${with_sc}">
+    <xacro:link_with_sc no_prefix="${no_prefix}" name="link7" gazebo="${gazebo}" rpy="0 0 ${pi/4}" with_sc="${with_sc}">
       <self_collision_geometries>
         <xacro:collision_capsule xyz="0 0 0.01" direction="z" radius="${0.04+safety_distance}" length="0.14" />
@@ -111,17 +113,17 @@
       </self_collision_geometries>
     </xacro:link_with_sc>
-    <joint name="${arm_id}_joint7" type="revolute">
+    <joint name="${prefix}joint7" type="revolute">
       <xacro:franka-kinematics name="joint7" config="${kinematics}" />
-      <parent link="${arm_id}_link6"/>
-      <child link="${arm_id}_link7"/>
+      <parent link="${prefix}link6"/>
+      <child link="${prefix}link7"/>
       <axis xyz="0 0 1"/>
       <xacro:franka-limits name="joint7" config="${joint_limits}" />
       <xacro:franka-dynamics name="joint7" config="${dynamics}" />
     </joint>
-    <link name="${arm_id}_link8"/>
-    <joint name="${arm_id}_joint8" type="fixed">
+    <link name="${prefix}link8"/>
+    <joint name="${prefix}joint8" type="fixed">
       <xacro:franka-kinematics name="joint8" config="${kinematics}" />
-      <parent link="${arm_id}_link7" />
-      <child link="${arm_id}_link8" />
+      <parent link="${prefix}link7" />
+      <child link="${prefix}link8" />
     </joint>
   </xacro:macro>

File: robots/common/franka_robot.xacro (robot description, xacro)
@@ -18,9 +18,11 @@
                       use_fake_hardware:=false
                       fake_sensor_commands:=false
-                      gazebo_effort:=false">
+                      gazebo_effort:=false
+                      no_prefix:='false'">
     <xacro:include filename="$(find franka_description)/robots/common/utils.xacro" />
     <xacro:include filename="$(find franka_description)/robots/common/franka_arm.xacro" />
     <xacro:franka_arm
       arm_id="${arm_id}"
+      no_prefix="${no_prefix}"
       xyz="${xyz}"
       rpy="${rpy}"

File: robots/common/utils.xacro (robot description, xacro)
@@ -32,5 +32,6 @@
   <!-- self_collision_geometries:  self <collision> models        -->
   <!-- ========================================================== -->
-  <xacro:macro name="link_with_sc" params="name prefix=${arm_id}_ rpy:='0 0 0' **self_collision_geometries gazebo:=false with_sc:=false">
+  <xacro:macro name="link_with_sc" params="name no_prefix:='false' rpy:='0 0 0' **self_collision_geometries gazebo:=false with_sc:=false">
+    <xacro:property name="prefix" value="${'' if no_prefix else arm_id + '_'}" />
     <!-- sub-link defining detailed meshes for collision with environment -->
     <link name="${prefix}${name}">

File: robots/fer/fer.urdf.xacro (robot description, xacro)
@@ -2,4 +2,12 @@
 <robot xmlns:xacro="http://www.ros.org/wiki/xacro" name="fer">
   <xacro:include filename="$(find franka_description)/robots/common/franka_robot.xacro"/>
+  <!--
+    DEPRECATION NOTICE
+    argument arm_id is no longer supported and will be removed in the future.
+    This argument is ignored.
+  -->
+  <xacro:arg name="arm_id" default="fer" />
+  <!-- Don't print a prefix for joints, visuals, and links? -->
+  <xacro:arg name="no_prefix" default="false"/>
   <!-- Should an end-effector be mounted at the flange?" -->
   <xacro:arg name="hand" default="true" />
@@ -39,5 +47,6 @@
                       use_fake_hardware="$(arg use_fake_hardware)"
                       fake_sensor_commands="$(arg fake_sensor_commands)"
-                      gazebo_effort="$(arg gazebo_effort)">
+                      gazebo_effort="$(arg gazebo_effort)"
+                      no_prefix="$(arg no_prefix)">
   </xacro:franka_robot>
 </robot>

File: robots/fp3/fp3.urdf.xacro (robot description, xacro)
@@ -2,4 +2,12 @@
 <robot xmlns:xacro="http://www.ros.org/wiki/xacro" name="fp3">
   <xacro:include filename="$(find franka_description)/robots/common/franka_robot.xacro"/>
+  <!--
+    DEPRECATION NOTICE
+    argument arm_id is no longer supported and will be removed in the future.
+    This argument is ignored.
+  -->
+  <xacro:arg name="arm_id" default="fp3" />
+  <!-- Don't print a prefix for joints, visuals, and links? -->
+  <xacro:arg name="no_prefix" default="false"/>
   <!-- Should an end-effector be mounted at the flange?" -->
   <xacro:arg name="hand" default="true" />
@@ -33,5 +41,6 @@
                       use_fake_hardware="$(arg use_fake_hardware)"
                       fake_sensor_commands="$(arg fake_sensor_commands)"
-                      gazebo_effort="$(arg gazebo_effort)">
+                      gazebo_effort="$(arg gazebo_effort)"
+                      no_prefix="$(arg no_prefix)">
   </xacro:franka_robot>
 </robot>

File: robots/fr3/fr3.urdf.xacro (robot description, xacro)
@@ -2,4 +2,12 @@
 <robot xmlns:xacro="http://www.ros.org/wiki/xacro" name="fr3">
   <xacro:include filename="$(find franka_description)/robots/common/franka_robot.xacro"/>
+  <!--
+    DEPRECATION NOTICE
+    argument arm_id is no longer supported and will be removed in the future.
+    This argument is ignored.
+  -->
+  <xacro:arg name="arm_id" default="fr3" />
+  <!-- Don't print a prefix for joints, visuals, and links? -->
+  <xacro:arg name="no_prefix" default="false"/>
   <!-- Should an end-effector be mounted at the flange?" -->
   <xacro:arg name="hand" default="true" />
@@ -33,5 +41,6 @@
                       use_fake_hardware="$(arg use_fake_hardware)"
                       fake_sensor_commands="$(arg fake_sensor_commands)"
-                      gazebo_effort="$(arg gazebo_effort)">
+                      gazebo_effort="$(arg gazebo_effort)"
+                      no_prefix="$(arg no_prefix)">
   </xacro:franka_robot>
 </robot>
