Commit message: feat: support gazebo simulation in ros2

File: robots/common/franka_arm.ros2_control.xacro (robot description, xacro)
@@ -1,25 +1,31 @@
 <?xml version="1.0"?>
 <robot xmlns:xacro="http://www.ros.org/wiki/xacro">
-  <xacro:macro name="franka_arm_ros2_control" params="arm_id robot_ip use_fake_hardware:=^|false fake_sensor_commands:=^|false">
-    <ros2_control name="FrankaHardwareInterface" type="system">
-      <hardware>
-        <param name="arm_id">${arm_id}</param>
-        <xacro:if value="${use_fake_hardware}">
-          <plugin>fake_components/GenericSystem</plugin>
-          <param name="fake_sensor_commands">${fake_sensor_commands}</param>
-          <param name="state_following_offset">0.0</param>
-        </xacro:if>
-        <xacro:unless value="${use_fake_hardware}">
-          <plugin>franka_hardware/FrankaHardwareInterface</plugin>
-          <param name="robot_ip">${robot_ip}</param>
-        </xacro:unless>
-      </hardware>
+  <xacro:macro name="franka_arm_ros2_control" params="arm_id robot_ip use_fake_hardware:=^|false fake_sensor_commands:=^|false gazebo:=^|false hand:=^|false">
+      <ros2_control name="FrankaHardwareInterface" type="system">
+        <hardware>
+          <param name="arm_id">${arm_id}</param>
+          <xacro:if value="${use_fake_hardware}">
+            <plugin>fake_components/GenericSystem</plugin>
+            <param name="fake_sensor_commands">${fake_sensor_commands}</param>
+            <param name="state_following_offset">0.0</param>
+          </xacro:if>
+          <xacro:if value="${gazebo}">
+            <plugin>ign_ros2_control/IgnitionSystem</plugin>
+          </xacro:if>
+          <xacro:if value="${use_fake_hardware == 0 and gazebo == 0}">
+            <plugin>franka_hardware/FrankaHardwareInterface</plugin>
+            <param name="robot_ip">${robot_ip}</param>
+          </xacro:if>
+        </hardware>
       <xacro:macro name="configure_joint" params="joint_name initial_position">
         <joint name="${joint_name}">
-          <param name="initial_position">${initial_position}</param>
-          <command_interface name="effort"/>
+          <xacro:unless value="${gazebo}">
+            <command_interface name="effort"/>
+          </xacro:unless>
           <command_interface name="velocity"/>
           <command_interface name="position"/>
-          <state_interface name="position"/>
+          <state_interface name="position">
+            <param name="initial_value">${initial_position}</param>
+          </state_interface>
           <state_interface name="velocity"/>
           <state_interface name="effort"/>
@@ -33,5 +39,15 @@
       <xacro:configure_joint joint_name="${arm_id}_joint6" initial_position="${pi/2}"/>
       <xacro:configure_joint joint_name="${arm_id}_joint7" initial_position="${pi/4}"/>
+      <xacro:if value="${gazebo and hand}">
+        <xacro:configure_joint joint_name="${arm_id}_finger_joint1" initial_position="0.0" />
+      </xacro:if>
     </ros2_control>
+    <xacro:if value="${gazebo}">
+      <gazebo>
+        <plugin filename="ign_ros2_control-system" name="ign_ros2_control::IgnitionROS2ControlPlugin">
+          <parameters>$(find franka_gazebo_bringup)/config/franka_gazebo_controllers.yaml</parameters>
+        </plugin>
+      </gazebo>
+    </xacro:if>
   </xacro:macro>
 </robot>

File: robots/common/franka_robot.xacro (robot description, xacro)
@@ -1,5 +1,21 @@
 <?xml version='1.0' encoding='utf-8'?>
 <robot xmlns:xacro="http://www.ros.org/wiki/xacro">
-  <xacro:macro name="franka_robot" params="arm_id joint_limits kinematics inertials dynamics parent:='world' xyz:='0 0 0' rpy:='0 0 0' hand:='true' ee_id:=none gazebo:='false' with_sc:='false' ros2_control:=false robot_ip:='' use_fake_hardware:=false fake_sensor_commands:=false">
+  <xacro:macro name="franka_robot"
+              params="arm_id
+                      joint_limits
+                      kinematics
+                      inertials
+                      dynamics
+                      parent:='world'
+                      xyz:='0 0 0'
+                      rpy:='0 0 0'
+                      hand:='true'
+                      ee_id:=none
+                      gazebo:='false'
+                      with_sc:='false'
+                      ros2_control:=false
+                      robot_ip:=''
+                      use_fake_hardware:=false
+                      fake_sensor_commands:=false">
     <xacro:include filename="$(find franka_description)/robots/common/utils.xacro" />
     <xacro:include filename="$(find franka_description)/robots/common/franka_arm.xacro" />
@@ -109,5 +125,12 @@
     <xacro:if value="${ros2_control}">
       <xacro:include filename="$(find franka_description)/robots/common/franka_arm.ros2_control.xacro"/>
-      <xacro:franka_arm_ros2_control arm_id="$(arg arm_id)" robot_ip="$(arg robot_ip)" use_fake_hardware="$(arg use_fake_hardware)" fake_sensor_commands="$(arg fake_sensor_commands)"/>
+      <xacro:franka_arm_ros2_control
+          arm_id="$(arg arm_id)"
+          robot_ip="$(arg robot_ip)"
+          use_fake_hardware="$(arg use_fake_hardware)"
+          fake_sensor_commands="$(arg fake_sensor_commands)"
+          gazebo="$(arg gazebo)"
+          hand="$(arg hand)"
+      />
     </xacro:if>
   </xacro:macro>

Commit message: add: gazebo simulation joint friction and gazebo effort interface param

File: robots/common/franka_arm.ros2_control.xacro (robot description, xacro)
@@ -1,6 +1,13 @@
 <?xml version="1.0"?>
 <robot xmlns:xacro="http://www.ros.org/wiki/xacro">
-  <xacro:macro name="franka_arm_ros2_control" params="arm_id robot_ip use_fake_hardware:=^|false fake_sensor_commands:=^|false gazebo:=^|false hand:=^|false">
-      <ros2_control name="FrankaHardwareInterface" type="system">
+<xacro:macro name="franka_arm_ros2_control"
+         params="arm_id
+             robot_ip
+             use_fake_hardware:=^|false
+             fake_sensor_commands:=^|false
+             gazebo:=^|false
+             hand:=^|false
+             gazebo_effort:=^|false">
+    <ros2_control name="FrankaHardwareInterface" type="system">
         <hardware>
           <param name="arm_id">${arm_id}</param>
@@ -20,7 +27,11 @@
       <xacro:macro name="configure_joint" params="joint_name initial_position">
         <joint name="${joint_name}">
-          <xacro:unless value="${gazebo}">
+          <!--
+            deactivated for gazebo velocity and position interface due to a bug
+            https://github.com/ros-controls/gz_ros2_control/issues/343
+          -->
+          <xacro:if value="${gazebo == 0 or gazebo_effort == 1}">
             <command_interface name="effort"/>
-          </xacro:unless>
+          </xacro:if>
           <command_interface name="velocity"/>
           <command_interface name="position"/>

File: robots/common/franka_robot.xacro (robot description, xacro)
@@ -17,5 +17,6 @@
                       robot_ip:=''
                       use_fake_hardware:=false
-                      fake_sensor_commands:=false">
+                      fake_sensor_commands:=false
+                      gazebo_effort:=false">
     <xacro:include filename="$(find franka_description)/robots/common/utils.xacro" />
     <xacro:include filename="$(find franka_description)/robots/common/franka_arm.xacro" />
@@ -132,4 +133,5 @@
           gazebo="$(arg gazebo)"
           hand="$(arg hand)"
+          gazebo_effort="$(arg gazebo_effort)"
       />
     </xacro:if>

File: robots/fer/fer.urdf.xacro (robot description, xacro)
@@ -26,4 +26,6 @@
   <!-- Should fake sensors be used? -->
   <xacro:arg name="fake_sensor_commands" default="false" />
+  <!-- Should the robot be spawned in Gazebo with effort interfaces?" -->
+  <xacro:arg name="gazebo_effort" default="false" />
   <xacro:franka_robot arm_id="$(arg arm_id)"
                       joint_limits="${xacro.load_yaml('$(find franka_description)/robots/$(arg arm_id)/joint_limits.yaml')}"
@@ -39,4 +41,4 @@
                       use_fake_hardware="$(arg use_fake_hardware)"
                       fake_sensor_commands="$(arg fake_sensor_commands)"
-                      />
+                      gazebo_effort="$(arg gazebo_effort)">
 </robot>

File: robots/fp3/fp3.urdf.xacro (robot description, xacro)
@@ -20,4 +20,6 @@
   <!-- Should the robot be spawned in Gazebo?" -->
   <xacro:arg name="gazebo" default="false" />
+  <!-- Should the robot be spawned in Gazebo with effort interfaces?" -->
+  <xacro:arg name="gazebo_effort" default="false" />
   <xacro:franka_robot arm_id="$(arg arm_id)"
                       joint_limits="${xacro.load_yaml('$(find franka_description)/robots/$(arg arm_id)/joint_limits.yaml')}"
@@ -32,5 +34,6 @@
                       robot_ip="$(arg robot_ip)"
                       use_fake_hardware="$(arg use_fake_hardware)"
-                      fake_sensor_commands="$(arg fake_sensor_commands)">
+                      fake_sensor_commands="$(arg fake_sensor_commands)"
+                      gazebo_effort="$(arg gazebo_effort)">
   </xacro:franka_robot>
 </robot>

File: robots/fr3/fr3.urdf.xacro (robot description, xacro)
@@ -20,4 +20,6 @@
   <!-- Should the robot be spawned in Gazebo?" -->
   <xacro:arg name="gazebo" default="false" />
+  <!-- Should the robot be spawned in Gazebo with effort interfaces?" -->
+  <xacro:arg name="gazebo_effort" default="false" />
   <xacro:franka_robot arm_id="$(arg arm_id)"
                       joint_limits="${xacro.load_yaml('$(find franka_description)/robots/$(arg arm_id)/joint_limits.yaml')}"
@@ -32,5 +34,6 @@
                       robot_ip="$(arg robot_ip)"
                       use_fake_hardware="$(arg use_fake_hardware)"
-                      fake_sensor_commands="$(arg fake_sensor_commands)">
+                      fake_sensor_commands="$(arg fake_sensor_commands)"
+                      gazebo_effort="$(arg gazebo_effort)">
   </xacro:franka_robot>
 </robot>

Commit message: feat: Adding the .xacro definition for dual arm setups

File: robots/common/franka_arm.ros2_control.xacro (robot description, xacro)
@@ -8,8 +8,11 @@
              gazebo:=^|false
              hand:=^|false
-             gazebo_effort:=^|false">
-    <ros2_control name="FrankaHardwareInterface" type="system">
+             gazebo_effort:=^|false
+             arm_prefix:=''">
+    <xacro:property name="prefix" value="${'' if arm_prefix == '' else arm_prefix + '_'}" />
+    <ros2_control name="${prefix}FrankaHardwareInterface" type="system">
         <hardware>
           <param name="arm_id">${arm_id}</param>
+          <param name="prefix">${prefix}</param>
           <xacro:if value="${use_fake_hardware}">
             <plugin>fake_components/GenericSystem</plugin>
@@ -23,4 +26,5 @@
             <plugin>franka_hardware/FrankaHardwareInterface</plugin>
             <param name="robot_ip">${robot_ip}</param>
+            <param name="arm_prefix">${arm_prefix}</param>
           </xacro:if>
         </hardware>
@@ -44,11 +48,11 @@
         </joint>
       </xacro:macro>
-      <xacro:configure_joint joint_name="${arm_id}_joint1" initial_position="0.0"/>
-      <xacro:configure_joint joint_name="${arm_id}_joint2" initial_position="${-pi/4}"/>
-      <xacro:configure_joint joint_name="${arm_id}_joint3" initial_position="0.0"/>
-      <xacro:configure_joint joint_name="${arm_id}_joint4" initial_position="${-3*pi/4}"/>
-      <xacro:configure_joint joint_name="${arm_id}_joint5" initial_position="0.0"/>
-      <xacro:configure_joint joint_name="${arm_id}_joint6" initial_position="${pi/2}"/>
-      <xacro:configure_joint joint_name="${arm_id}_joint7" initial_position="${pi/4}"/>
+      <xacro:configure_joint joint_name="${prefix}${arm_id}_joint1" initial_position="0.0"/>
+      <xacro:configure_joint joint_name="${prefix}${arm_id}_joint2" initial_position="${-pi/4}"/>
+      <xacro:configure_joint joint_name="${prefix}${arm_id}_joint3" initial_position="0.0"/>
+      <xacro:configure_joint joint_name="${prefix}${arm_id}_joint4" initial_position="${-3*pi/4}"/>
+      <xacro:configure_joint joint_name="${prefix}${arm_id}_joint5" initial_position="0.0"/>
+      <xacro:configure_joint joint_name="${prefix}${arm_id}_joint6" initial_position="${pi/2}"/>
+      <xacro:configure_joint joint_name="${prefix}${arm_id}_joint7" initial_position="${pi/4}"/>
       <xacro:if value="${gazebo and hand}">
         <xacro:configure_joint joint_name="${arm_id}_finger_joint1" initial_position="0.0" />

File: robots/common/franka_arm.xacro (robot description, xacro)
@@ -8,7 +8,7 @@
   <!-- inertials: description of the inertials that comes from a YAML file. Example definition: ${xacro.load_yaml('$(find franka_description)/robots/fr3/inertials.yaml')} -->
   <!-- dynamics: description of the dynamics that comes from a YAML file. Example definition: ${xacro.load_yaml('$(find franka_description)/robots/fr3/dynamics.yaml')} -->
-  <xacro:macro name="franka_arm" params="arm_id no_prefix:=false description_pkg:='franka_description' connected_to:='base' xyz:='0 0 0' rpy:='0 0 0' gazebo:='false' safety_distance:=0 joint_limits inertials kinematics dynamics with_sc:=false" >
-    <!-- Define a property that defaults to 'arm_id' concatenated with an underscore if 'no_prefix' is not set -->
-    <xacro:property name="prefix" value="${'' if no_prefix else arm_id + '_'}" />
+  <xacro:macro name="franka_arm" params="arm_id arm_prefix:='' no_prefix:=false description_pkg:='franka_description' connected_to:='base' xyz:='0 0 0' rpy:='0 0 0' gazebo:='false' safety_distance:=0 joint_limits inertials kinematics dynamics with_sc:=false" >
+    <!-- Define a property that defaults to 'arm_prefix_arm_id' concatenated with an underscore if 'no_prefix' is not set -->
+    <xacro:property name="prefix" value="${'' if no_prefix else arm_prefix + arm_id + '_'}" />
     <xacro:if value="${gazebo}">
       <xacro:property name="connected_to" value="" />
@@ -17,5 +17,5 @@
       <link name="${connected_to}">
       </link>
-      <joint name="${connected_to}_joint" type="fixed">
+      <joint name="${prefix}${connected_to}_joint" type="fixed">
         <parent link="${connected_to}"/>
         <child link="${prefix}link0"/>

File: robots/common/franka_robot.xacro (robot description, xacro)
@@ -19,9 +19,12 @@
                       fake_sensor_commands:=false
                       gazebo_effort:=false
-                      no_prefix:='false'">
+                      no_prefix:='false'
+                      arm_prefix:=''
+                      connected_to:='base'">
     <xacro:include filename="$(find franka_description)/robots/common/utils.xacro" />
     <xacro:include filename="$(find franka_description)/robots/common/franka_arm.xacro" />
     <xacro:franka_arm
       arm_id="${arm_id}"
+      arm_prefix="${arm_prefix}"
       no_prefix="${no_prefix}"
       xyz="${xyz}"
@@ -34,4 +37,5 @@
       dynamics="${dynamics}"
       with_sc="${with_sc}"
+      connected_to="${connected_to}"
     />
     <xacro:if value="${hand and ee_id == 'franka_hand'}">
@@ -129,6 +133,6 @@
       <xacro:include filename="$(find franka_description)/robots/common/franka_arm.ros2_control.xacro"/>
       <xacro:franka_arm_ros2_control
-          arm_id="$(arg arm_id)"
-          robot_ip="$(arg robot_ip)"
+          arm_id="${arm_id}"
+          robot_ip="${robot_ip}"
           use_fake_hardware="$(arg use_fake_hardware)"
           fake_sensor_commands="$(arg fake_sensor_commands)"
@@ -136,4 +140,5 @@
           hand="$(arg hand)"
           gazebo_effort="$(arg gazebo_effort)"
+          arm_prefix="${arm_prefix}"
       />
     </xacro:if>

File: robots/common/utils.xacro (robot description, xacro)
@@ -33,5 +33,5 @@
   <!-- ========================================================== -->
   <xacro:macro name="link_with_sc" params="name no_prefix:='false' rpy:='0 0 0' **self_collision_geometries gazebo:=false with_sc:=false">
-    <xacro:property name="prefix" value="${'' if no_prefix else arm_id + '_'}" />
+    <xacro:property name="prefix" value="${'' if no_prefix else arm_prefix + arm_id + '_'}" />
     <!-- sub-link defining detailed meshes for collision with environment -->
     <link name="${prefix}${name}">
@@ -157,20 +157,20 @@
   <!-- ========================================================== -->
   <xacro:macro name="transmission-franka-state" params="arm_id:=fer">
-    <transmission name="${arm_id}_franka_state">
+    <transmission name="${arm_prefix}${arm_id}_franka_state">
       <type>franka_hw/FrankaStateInterface</type>
-      <joint name="${arm_id}_joint1"><hardwareInterface>franka_hw/FrankaStateInterface</hardwareInterface></joint>
-      <joint name="${arm_id}_joint2"><hardwareInterface>franka_hw/FrankaStateInterface</hardwareInterface></joint>
-      <joint name="${arm_id}_joint3"><hardwareInterface>franka_hw/FrankaStateInterface</hardwareInterface></joint>
-      <joint name="${arm_id}_joint4"><hardwareInterface>franka_hw/FrankaStateInterface</hardwareInterface></joint>
-      <joint name="${arm_id}_joint5"><hardwareInterface>franka_hw/FrankaStateInterface</hardwareInterface></joint>
-      <joint name="${arm_id}_joint6"><hardwareInterface>franka_hw/FrankaStateInterface</hardwareInterface></joint>
-      <joint name="${arm_id}_joint7"><hardwareInterface>franka_hw/FrankaStateInterface</hardwareInterface></joint>
-      <actuator name="${arm_id}_motor1"><hardwareInterface>franka_hw/FrankaStateInterface</hardwareInterface></actuator>
-      <actuator name="${arm_id}_motor2"><hardwareInterface>franka_hw/FrankaStateInterface</hardwareInterface></actuator>
-      <actuator name="${arm_id}_motor3"><hardwareInterface>franka_hw/FrankaStateInterface</hardwareInterface></actuator>
-      <actuator name="${arm_id}_motor4"><hardwareInterface>franka_hw/FrankaStateInterface</hardwareInterface></actuator>
-      <actuator name="${arm_id}_motor5"><hardwareInterface>franka_hw/FrankaStateInterface</hardwareInterface></actuator>
-      <actuator name="${arm_id}_motor6"><hardwareInterface>franka_hw/FrankaStateInterface</hardwareInterface></actuator>
-      <actuator name="${arm_id}_motor7"><hardwareInterface>franka_hw/FrankaStateInterface</hardwareInterface></actuator>
+      <joint name="${arm_prefix}${arm_id}_joint1"><hardwareInterface>franka_hw/FrankaStateInterface</hardwareInterface></joint>
+      <joint name="${arm_prefix}${arm_id}_joint2"><hardwareInterface>franka_hw/FrankaStateInterface</hardwareInterface></joint>
+      <joint name="${arm_prefix}${arm_id}_joint3"><hardwareInterface>franka_hw/FrankaStateInterface</hardwareInterface></joint>
+      <joint name="${arm_prefix}${arm_id}_joint4"><hardwareInterface>franka_hw/FrankaStateInterface</hardwareInterface></joint>
+      <joint name="${arm_prefix}${arm_id}_joint5"><hardwareInterface>franka_hw/FrankaStateInterface</hardwareInterface></joint>
+      <joint name="${arm_prefix}${arm_id}_joint6"><hardwareInterface>franka_hw/FrankaStateInterface</hardwareInterface></joint>
+      <joint name="${arm_prefix}${arm_id}_joint7"><hardwareInterface>franka_hw/FrankaStateInterface</hardwareInterface></joint>
+      <actuator name="${arm_prefix}${arm_id}_motor1"><hardwareInterface>franka_hw/FrankaStateInterface</hardwareInterface></actuator>
+      <actuator name="${arm_prefix}${arm_id}_motor2"><hardwareInterface>franka_hw/FrankaStateInterface</hardwareInterface></actuator>
+      <actuator name="${arm_prefix}${arm_id}_motor3"><hardwareInterface>franka_hw/FrankaStateInterface</hardwareInterface></actuator>
+      <actuator name="${arm_prefix}${arm_id}_motor4"><hardwareInterface>franka_hw/FrankaStateInterface</hardwareInterface></actuator>
+      <actuator name="${arm_prefix}${arm_id}_motor5"><hardwareInterface>franka_hw/FrankaStateInterface</hardwareInterface></actuator>
+      <actuator name="${arm_prefix}${arm_id}_motor6"><hardwareInterface>franka_hw/FrankaStateInterface</hardwareInterface></actuator>
+      <actuator name="${arm_prefix}${arm_id}_motor7"><hardwareInterface>franka_hw/FrankaStateInterface</hardwareInterface></actuator>
     </transmission>
   </xacro:macro>
@@ -184,5 +184,5 @@
   <!-- ============================================================ -->
   <xacro:macro name="transmission-franka-model" params="arm_id:=fer root:=fer_joint1 tip:=fer_joint7">
-    <transmission name="${arm_id}_franka_model">
+    <transmission name="${arm_prefix}${arm_id}_franka_model">
       <type>franka_hw/FrankaModelInterface</type>
       <joint name="${root}">

File: robots/fer/fer.urdf.xacro (robot description, xacro)
@@ -48,5 +48,7 @@
                       fake_sensor_commands="$(arg fake_sensor_commands)"
                       gazebo_effort="$(arg gazebo_effort)"
-                      no_prefix="$(arg no_prefix)">
+                      no_prefix="$(arg no_prefix)"
+                      arm_prefix= ""
+                      connected_to= "base">
   </xacro:franka_robot>
 </robot>

File: robots/fp3/fp3.urdf.xacro (robot description, xacro)
@@ -42,5 +42,7 @@
                       fake_sensor_commands="$(arg fake_sensor_commands)"
                       gazebo_effort="$(arg gazebo_effort)"
-                      no_prefix="$(arg no_prefix)">
+                      no_prefix="$(arg no_prefix)"
+                      arm_prefix= ""
+                      connected_to= "base">
   </xacro:franka_robot>
 </robot>

File: robots/fr3/fr3.urdf.xacro (robot description, xacro)
@@ -42,5 +42,7 @@
                       fake_sensor_commands="$(arg fake_sensor_commands)"
                       gazebo_effort="$(arg gazebo_effort)"
-                      no_prefix="$(arg no_prefix)">
+                      no_prefix="$(arg no_prefix)"
+                      arm_prefix= ""
+                      connected_to= "base">
   </xacro:franka_robot>
 </robot>
