Commit message: fix: Fixed a wrong parameter name feat: Adapted the URDFs to use the 'multi arm' hardware interface in case of multi arm setups

File: robots/common/franka_arm.ros2_control.xacro (robot description, xacro)
@@ -9,10 +9,10 @@
              hand:=^|false
              gazebo_effort:=^|false
-             arm_prefix:=''">
-    <xacro:property name="prefix" value="${'' if arm_prefix == '' else arm_prefix + '_'}" />
-    <ros2_control name="${prefix}FrankaHardwareInterface" type="system">
+             arm_prefix:=''
+             multi_arm:=false">
+    <ros2_control name="${arm_prefix}FrankaHardwareInterface" type="system">
         <hardware>
           <param name="arm_id">${arm_id}</param>
-          <param name="prefix">${prefix}</param>
+          <param name="prefix">${arm_prefix}</param>
           <xacro:if value="${use_fake_hardware}">
             <plugin>fake_components/GenericSystem</plugin>
@@ -23,6 +23,11 @@
             <plugin>franka_ign_ros2_control/IgnitionSystem</plugin>
           </xacro:if>
-          <xacro:if value="${use_fake_hardware == 0 and gazebo == 0}">
+          <xacro:if value="${use_fake_hardware == 0 and gazebo == 0 and multi_arm == 0}">
             <plugin>franka_hardware/FrankaHardwareInterface</plugin>
+            <param name="robot_ip">${robot_ip}</param>
+            <param name="arm_prefix">${arm_prefix}</param>
+          </xacro:if>
+          <xacro:if value="${use_fake_hardware == 0 and gazebo == 0 and multi_arm == 1}">
+            <plugin>franka_hardware/MultiFrankaHardwareInterface</plugin>
             <param name="robot_ip">${robot_ip}</param>
             <param name="arm_prefix">${arm_prefix}</param>
@@ -34,10 +39,13 @@
             deactivated for gazebo velocity and position interface due to a bug
             https://github.com/ros-controls/gz_ros2_control/issues/343
-          -->
+            Command Interfaces -->
+          <xacro:if value="${multi_arm == 0}">
+            <command_interface name="position"/>
+          </xacro:if>
+          <command_interface name="velocity"/>
           <xacro:if value="${gazebo == 0 or gazebo_effort == 1}">
             <command_interface name="effort"/>
           </xacro:if>
-          <command_interface name="velocity"/>
-          <command_interface name="position"/>
+          <!-- State Interfaces -->
           <state_interface name="position">
             <param name="initial_value">${initial_position}</param>
@@ -48,11 +56,11 @@
         </joint>
       </xacro:macro>
-      <xacro:configure_joint joint_name="${prefix}${arm_id}_joint1" initial_position="0.0"/>
-      <xacro:configure_joint joint_name="${prefix}${arm_id}_joint2" initial_position="${-pi/4}"/>
-      <xacro:configure_joint joint_name="${prefix}${arm_id}_joint3" initial_position="0.0"/>
-      <xacro:configure_joint joint_name="${prefix}${arm_id}_joint4" initial_position="${-3*pi/4}"/>
-      <xacro:configure_joint joint_name="${prefix}${arm_id}_joint5" initial_position="0.0"/>
-      <xacro:configure_joint joint_name="${prefix}${arm_id}_joint6" initial_position="${pi/2}"/>
-      <xacro:configure_joint joint_name="${prefix}${arm_id}_joint7" initial_position="${pi/4}"/>
+      <xacro:configure_joint joint_name="${arm_prefix}${arm_id}_joint1" initial_position="0.0"/>
+      <xacro:configure_joint joint_name="${arm_prefix}${arm_id}_joint2" initial_position="${-pi/4}"/>
+      <xacro:configure_joint joint_name="${arm_prefix}${arm_id}_joint3" initial_position="0.0"/>
+      <xacro:configure_joint joint_name="${arm_prefix}${arm_id}_joint4" initial_position="${-3*pi/4}"/>
+      <xacro:configure_joint joint_name="${arm_prefix}${arm_id}_joint5" initial_position="0.0"/>
+      <xacro:configure_joint joint_name="${arm_prefix}${arm_id}_joint6" initial_position="${pi/2}"/>
+      <xacro:configure_joint joint_name="${arm_prefix}${arm_id}_joint7" initial_position="${pi/4}"/>
       <xacro:if value="${gazebo and hand}">
         <xacro:configure_joint joint_name="${arm_id}_finger_joint1" initial_position="0.0" />

File: robots/common/franka_robot.xacro (robot description, xacro)
@@ -21,5 +21,6 @@
                       no_prefix:='false'
                       arm_prefix:=''
-                      connected_to:='base'">
+                      connected_to:='base'
+                      multi_arm:=false">
     <xacro:include filename="$(find franka_description)/robots/common/utils.xacro" />
     <xacro:include filename="$(find franka_description)/robots/common/franka_arm.xacro" />
@@ -147,4 +148,5 @@
           gazebo_effort="$(arg gazebo_effort)"
           arm_prefix="${arm_prefix}"
+          multi_arm="$(arg multi_arm)"
       />
     </xacro:if>

File: robots/fer/fer.urdf.xacro (robot description, xacro)
@@ -34,4 +34,6 @@
   <!-- Should the robot be spawned in Gazebo with effort interfaces?" -->
   <xacro:arg name="gazebo_effort" default="false" />
+  <!-- For a multi arm setup, we need a threaded robot running async-->
+  <xacro:arg name="multi_arm" default="false" />
   <xacro:franka_robot arm_id="fer"
                       joint_limits="${xacro.load_yaml('$(find franka_description)/robots/fer/joint_limits.yaml')}"

File: robots/fp3/fp3.urdf.xacro (robot description, xacro)
@@ -28,4 +28,6 @@
   <!-- Should the robot be spawned in Gazebo with effort interfaces?" -->
   <xacro:arg name="gazebo_effort" default="false" />
+  <!-- For a multi arm setup, we need a threaded robot running async-->
+  <xacro:arg name="multi_arm" default="false" />
   <xacro:franka_robot arm_id="fp3"
                       joint_limits="${xacro.load_yaml('$(find franka_description)/robots/fp3/joint_limits.yaml')}"

File: robots/fr3/fr3.urdf.xacro (robot description, xacro)
@@ -28,4 +28,6 @@
   <!-- Should the robot be spawned in Gazebo with effort interfaces?" -->
   <xacro:arg name="gazebo_effort" default="false" />
+  <!-- For a multi arm setup, we need a threaded robot running async-->
+  <xacro:arg name="multi_arm" default="false" />
   <xacro:franka_robot arm_id="fr3"
                       joint_limits="${xacro.load_yaml('$(find franka_description)/robots/fr3/joint_limits.yaml')}"

File: robots/multi_arm/multi_arm.urdf.xacro (robot description, xacro)
@@ -12,9 +12,9 @@
   <xacro:arg name="number_of_robots" default = "2"/>
   <!-- Define arguments -->
-  <xacro:arg name="xyz" default="['0 0.1 0','0 -0.1 0']" />
-  <xacro:property name="xyz_list" value="${$(arg xyz)}" />
+  <xacro:arg name="xyz_values" default="['0 0.1 0','0 -0.1 0']" />
+  <xacro:property name="xyz_list" value="${$(arg xyz_values)}" />
   <!-- Define arguments -->
-  <xacro:arg name="rpy" default="['-0.7 0 0','0.7 0 0']" />
-  <xacro:property name="rpy_list" value="${$(arg rpy)}" />
+  <xacro:arg name="rpy_values" default="['-0.7 0 0','0.7 0 0']" />
+  <xacro:property name="rpy_list" value="${$(arg rpy_values)}" />
   <!-- Don't print a prefix for joints, visuals, and links? -->
   <xacro:arg name="no_prefix" default="false"/>
@@ -42,6 +42,9 @@
   <xacro:arg name="arm_prefixes" default="['left','right']" />
   <xacro:property name="arm_prefixes_list" value="${$(arg arm_prefixes)}" />
+  <!-- For a multi arm setup, we need a threaded robot running async-->
+  <xacro:arg name="multi_arm" default="true" />
   <link name="base">
   </link>
+  <!-- The multi robot setup configures 'multi_arm' by default to true s.t. it uses the async threading approach for the hardware interface -->
   <xacro:macro name="loop" params="i">
     <xacro:unless value="${i == $(arg number_of_robots)}">
@@ -67,5 +70,6 @@
                           no_prefix="$(arg no_prefix)"
                           arm_prefix= "${arm_prefixes_list[i]}_"
-                          connected_to="${arm_prefixes_list[i]}_base">
+                          connected_to="${arm_prefixes_list[i]}_base"
+                          multi_arm="$(arg multi_arm)">
       </xacro:franka_robot>
       <xacro:loop i="${i+1}"/>

Commit message: fix: underscore removed from arm prefix

File: robots/common/franka_arm.ros2_control.xacro (robot description, xacro)
@@ -11,5 +11,6 @@
              arm_prefix:=''
              multi_arm:=false">
-    <ros2_control name="${arm_prefix}FrankaHardwareInterface" type="system">
+    <xacro:property name="arm_prefix_modified" value="${'' if arm_prefix == '' else arm_prefix + '_'}" />
+    <ros2_control name="${arm_prefix_modified}FrankaHardwareInterface" type="system">
         <hardware>
           <param name="arm_id">${arm_id}</param>
@@ -56,11 +57,11 @@
         </joint>
       </xacro:macro>
-      <xacro:configure_joint joint_name="${arm_prefix}${arm_id}_joint1" initial_position="0.0"/>
-      <xacro:configure_joint joint_name="${arm_prefix}${arm_id}_joint2" initial_position="${-pi/4}"/>
-      <xacro:configure_joint joint_name="${arm_prefix}${arm_id}_joint3" initial_position="0.0"/>
-      <xacro:configure_joint joint_name="${arm_prefix}${arm_id}_joint4" initial_position="${-3*pi/4}"/>
-      <xacro:configure_joint joint_name="${arm_prefix}${arm_id}_joint5" initial_position="0.0"/>
-      <xacro:configure_joint joint_name="${arm_prefix}${arm_id}_joint6" initial_position="${pi/2}"/>
-      <xacro:configure_joint joint_name="${arm_prefix}${arm_id}_joint7" initial_position="${pi/4}"/>
+      <xacro:configure_joint joint_name="${arm_prefix_modified}${arm_id}_joint1" initial_position="0.0"/>
+      <xacro:configure_joint joint_name="${arm_prefix_modified}${arm_id}_joint2" initial_position="${-pi/4}"/>
+      <xacro:configure_joint joint_name="${arm_prefix_modified}${arm_id}_joint3" initial_position="0.0"/>
+      <xacro:configure_joint joint_name="${arm_prefix_modified}${arm_id}_joint4" initial_position="${-3*pi/4}"/>
+      <xacro:configure_joint joint_name="${arm_prefix_modified}${arm_id}_joint5" initial_position="0.0"/>
+      <xacro:configure_joint joint_name="${arm_prefix_modified}${arm_id}_joint6" initial_position="${pi/2}"/>
+      <xacro:configure_joint joint_name="${arm_prefix_modified}${arm_id}_joint7" initial_position="${pi/4}"/>
       <xacro:if value="${gazebo and hand}">
         <xacro:configure_joint joint_name="${arm_id}_finger_joint1" initial_position="0.0" />

File: robots/common/franka_robot.xacro (robot description, xacro)
@@ -25,7 +25,8 @@
     <xacro:include filename="$(find franka_description)/robots/common/utils.xacro" />
     <xacro:include filename="$(find franka_description)/robots/common/franka_arm.xacro" />
+    <xacro:property name="arm_prefix_modified" value="${'' if arm_prefix == '' else arm_prefix + '_'}" />
     <xacro:franka_arm
       arm_id="${arm_id}"
-      arm_prefix="${arm_prefix}"
+      arm_prefix="${arm_prefix_modified}"
       no_prefix="${no_prefix}"
       xyz="${xyz}"
@@ -53,7 +54,7 @@
       <xacro:property name="connection" value="${special_connection if special_connection != '' else arm_id + '_link8'}" />
       <xacro:franka_hand
-        connected_to="${arm_prefix}${connection}"
+        connected_to="${arm_prefix_modified}${connection}"
         arm_id="${arm_id}"
-        arm_prefix="${arm_prefix}"
+        arm_prefix="${arm_prefix_modified}"
         ee_id="${ee_id}_${ee_color}"
         ee_inertials="${xacro.load_yaml('$(find franka_description)/end_effectors/$(arg ee_id)/inertials.yaml')}"
@@ -75,7 +76,7 @@
       <xacro:property name="connection" value="${special_connection if special_connection == '' else arm_id + '_link8'}" />
       <xacro:ee_with_one_link
-        connected_to="${arm_prefix}${connection}"
+        connected_to="${arm_prefix_modified}${connection}"
         arm_id="${arm_id}"
-        arm_prefix="${arm_prefix}"
+        arm_prefix="${arm_prefix_modified}"
         ee_id="${ee_id}"
         ee_inertials="${xacro.load_yaml('$(find franka_description)/end_effectors/$(arg ee_id)/inertials.yaml')}"

File: robots/multi_arm/multi_arm.urdf.xacro (robot description, xacro)
@@ -69,5 +69,5 @@
                           gazebo_effort="$(arg gazebo_effort)"
                           no_prefix="$(arg no_prefix)"
-                          arm_prefix= "${arm_prefixes_list[i]}_"
+                          arm_prefix= "${arm_prefixes_list[i]}"
                           connected_to="${arm_prefixes_list[i]}_base"
                           multi_arm="$(arg multi_arm)">
