Commit message: fix: robot model does not need to be specified for ee urdf

File: end_effectors/common/ee_with_one_link.xacro (robot description, xacro)
@@ -3,8 +3,12 @@
   <!-- safety_distance: Minimum safety distance in [m] by which the collision volumes are expanded and which is enforced during robot motions -->
   <xacro:macro name="ee_with_one_link" params="connected_to:='' arm_id ee_id ee_inertials rpy:='0 0 0' xyz:='0 0 0' tcp_xyz:='0 0 0' tcp_rpy:='0 0 0' safety_distance:=0 gazebo:=false description_pkg:=franka_description with_sc:=false">
+    <xacro:property name="ee_prefix" default="robot_"/>
+    <xacro:unless value="${arm_id != ''}">
+      <xacro:property name="${ee_prefix}" value="${arm_id}" />
+    </xacro:unless>
     <xacro:unless value="${connected_to == ''}">
-      <joint name="${arm_id}_${ee_id}_joint" type="fixed">
+      <joint name="${ee_prefix}${ee_id}_joint" type="fixed">
         <parent link="${connected_to}" />
-        <child link="${arm_id}_${ee_id}" />
+        <child link="${ee_prefix}${ee_id}" />
         <origin xyz="${xyz}" rpy="${rpy}" />
       </joint>
@@ -17,9 +21,9 @@
     </xacro:ee_link_with_sc>
     <!-- Define the ${ee_id}_tcp frame -->
-    <link name="${arm_id}_${ee_id}_tcp" />
-    <joint name="${arm_id}_${ee_id}_tcp_joint" type="fixed">
+    <link name="${ee_prefix}${ee_id}_tcp" />
+    <joint name="${ee_prefix}${ee_id}_tcp_joint" type="fixed">
       <origin xyz="${tcp_xyz}" rpy="${tcp_rpy}" />
-      <parent link="${arm_id}_${ee_id}" />
-      <child link="${arm_id}_${ee_id}_tcp" />
+      <parent link="${ee_prefix}${ee_id}" />
+      <child link="${ee_prefix}${ee_id}_tcp" />
     </joint>
   </xacro:macro>

File: end_effectors/common/franka_hand.xacro (robot description, xacro)
@@ -3,8 +3,12 @@
   <!-- safety_distance: Minimum safety distance in [m] by which the collision volumes are expanded and which is enforced during robot motions -->
   <xacro:macro name="franka_hand" params="connected_to:='' arm_id ee_id ee_inertials rpy:='0 0 0' xyz:='0 0 0' tcp_xyz:='0 0 0.1034' tcp_rpy:='0 0 0' safety_distance:=0 gazebo:=false description_pkg:=franka_description with_sc:=false">
+    <xacro:property name="ee_prefix" default="robot_"/>
+    <xacro:unless value="${arm_id != ''}">
+      <xacro:property name="${ee_prefix}" value="${arm_id}" />
+    </xacro:unless>
     <xacro:unless value="${connected_to == ''}">
-      <joint name="${arm_id}_hand_joint" type="fixed">
+      <joint name="${ee_prefix}hand_joint" type="fixed">
         <parent link="${connected_to}" />
-        <child link="${arm_id}_hand" />
+        <child link="${ee_prefix}hand" />
         <origin xyz="${xyz}" rpy="${rpy}" />
       </joint>
@@ -17,12 +21,12 @@
     </xacro:ee_link_with_sc>
     <!-- Define the hand_tcp frame -->
-    <link name="${arm_id}_hand_tcp" />
-    <joint name="${arm_id}_hand_tcp_joint" type="fixed">
+    <link name="${ee_prefix}hand_tcp" />
+    <joint name="${ee_prefix}hand_tcp_joint" type="fixed">
       <origin xyz="${tcp_xyz}" rpy="${tcp_rpy}" />
-      <parent link="${arm_id}_hand" />
-      <child link="${arm_id}_hand_tcp" />
+      <parent link="${ee_prefix}hand" />
+      <child link="${ee_prefix}hand_tcp" />
     </joint>
-    <link name="${arm_id}_leftfinger">
-      <visual name="${arm_id}_leftfinger_visual">
+    <link name="${ee_prefix}leftfinger">
+      <visual name="${ee_prefix}leftfinger_visual">
         <geometry>
           <mesh filename="package://${description_pkg}/meshes/robot_ee/${ee_id}/visual/finger.dae" />
@@ -61,6 +65,6 @@
       </xacro:if>
     </link>
-    <link name="${arm_id}_rightfinger">
-      <visual name="${arm_id}_rightfinger_visual">
+    <link name="${ee_prefix}rightfinger">
+      <visual name="${ee_prefix}rightfinger_visual">
         <origin xyz="0 0 0" rpy="0 0 ${pi}" />
         <geometry>
@@ -100,7 +104,7 @@
       </xacro:if>
     </link>
-    <joint name="${arm_id}_finger_joint1" type="prismatic">
-      <parent link="${arm_id}_hand" />
-      <child link="${arm_id}_leftfinger" />
+    <joint name="${ee_prefix}finger_joint1" type="prismatic">
+      <parent link="${ee_prefix}hand" />
+      <child link="${ee_prefix}leftfinger" />
       <origin xyz="0 0 0.0584" rpy="0 0 0" />
       <axis xyz="0 1 0" />
@@ -108,11 +112,11 @@
       <dynamics damping="0.3" />
     </joint>
-    <joint name="${arm_id}_finger_joint2" type="prismatic">
-      <parent link="${arm_id}_hand" />
-      <child link="${arm_id}_rightfinger" />
+    <joint name="${ee_prefix}finger_joint2" type="prismatic">
+      <parent link="${ee_prefix}hand" />
+      <child link="${ee_prefix}rightfinger" />
       <origin xyz="0 0 0.0584" rpy="0 0 0" />
       <axis xyz="0 -1 0" />
       <limit effort="100" lower="0.0" upper="0.04" velocity="0.2" />
-      <mimic joint="${arm_id}_finger_joint1" />
+      <mimic joint="${ee_prefix}finger_joint1" />
       <dynamics damping="0.3" />
     </joint>

File: end_effectors/common/utils.xacro (robot description, xacro)
@@ -32,5 +32,5 @@
   <!-- self_collision_geometries:  self <collision> models        -->
   <!-- ========================================================== -->
-  <xacro:macro name="ee_link_with_sc" params="name prefix=${arm_id}_ rpy:='0 0 0' **self_collision_geometries gazebo:=false with_sc:=false">
+  <xacro:macro name="ee_link_with_sc" params="name prefix=${ee_prefix} rpy:='0 0 0' **self_collision_geometries gazebo:=false with_sc:=false">
     <!-- sub-link defining detailed meshes for collision with environment -->
     <link name="${prefix}${name}">
