Commit message: feat: Preparing changes for Gazebo

File: end_effectors/common/franka_hand.xacro (robot description, xacro)
@@ -58,5 +58,5 @@
       </collision>
       <xacro:if value="${gazebo}">
-        <xacro:franka-inertials name="leftfinger" />
+        <xacro:ee-inertials name="leftfinger" />
       </xacro:if>
     </link>
@@ -97,5 +97,5 @@
       </collision>
       <xacro:if value="${gazebo}">
-        <xacro:franka-inertials name="rightfinger" />
+        <xacro:ee-inertials name="rightfinger" />
       </xacro:if>
     </link>

File: robots/common/franka_arm.xacro (robot description, xacro)
@@ -8,9 +8,12 @@
   <!-- inertials: description of the inertials that comes from a YAML file. Example definition: ${xacro.load_yaml('$(find franka_description)/robots/fr3/inertials.yaml')} -->
   <!-- dynamics: description of the dynamics that comes from a YAML file. Example definition: ${xacro.load_yaml('$(find franka_description)/robots/fr3/dynamics.yaml')} -->
-  <xacro:macro name="franka_arm" params="arm_id description_pkg:='franka_description' connected_to:='base' xyz:='0 0 0' rpy:='0 0 0' gazebo:=false safety_distance:=0 joint_limits inertials kinematics dynamics with_sc:=false" >
+  <xacro:macro name="franka_arm" params="arm_id description_pkg:='franka_description' connected_to:='base' xyz:='0 0 0' rpy:='0 0 0' gazebo:='false' safety_distance:=0 joint_limits inertials kinematics dynamics with_sc:=false" >
+    <xacro:if value="${gazebo}">
+      <xacro:property name="connected_to" value="" />
+    </xacro:if>
     <xacro:unless value="${not connected_to}">
       <link name="${connected_to}">
       </link>
-      <joint name="${connected_to}" type="fixed">
+      <joint name="${connected_to}_joint" type="fixed">
         <parent link="${connected_to}"/>
         <child link="${arm_id}_link0"/>

File: robots/common/franka_robot.xacro (robot description, xacro)
@@ -1,9 +1,11 @@
 <?xml version='1.0' encoding='utf-8'?>
 <robot xmlns:xacro="http://www.ros.org/wiki/xacro">
-  <xacro:macro name="franka_robot" params="arm_id joint_limits kinematics inertials dynamics parent:='world' xyz:='0 0 0' rpy:='0 0 0' hand ee_id:=none gazebo:=false with_sc:='false' ros2_control:=false robot_ip:='' use_fake_hardware:=false fake_sensor_commands:=false">
+  <xacro:macro name="franka_robot" params="arm_id joint_limits kinematics inertials dynamics parent:='world' xyz:='0 0 0' rpy:='0 0 0' hand:='true' ee_id:=none gazebo:='false' with_sc:='false' ros2_control:=false robot_ip:='' use_fake_hardware:=false fake_sensor_commands:=false">
     <xacro:include filename="$(find franka_description)/robots/common/utils.xacro" />
     <xacro:include filename="$(find franka_description)/robots/common/franka_arm.xacro" />
     <xacro:franka_arm
       arm_id="${arm_id}"
+      xyz="${xyz}"
+      rpy="${rpy}"
       safety_distance="0.03"
       gazebo="${gazebo}"
@@ -97,5 +99,5 @@
          tip="${arm_id}_joint8"
        />
-      <xacro:if value="${ee_id == franka_hand}">
+      <xacro:if value="${ee_id == 'franka_hand'}">
         <xacro:gazebo-joint joint="${arm_id}_finger_joint1" transmission="hardware_interface/EffortJointInterface" />
         <xacro:gazebo-joint joint="${arm_id}_finger_joint2" transmission="hardware_interface/EffortJointInterface" />
@@ -104,11 +106,4 @@
         <xacro:gazebo-friction link="${arm_id}_rightfinger" mu="1.13" />
       </xacro:if>
-      <gazebo>
-        <plugin name="gazebo_ros_control" filename="libgazebo_ros_control.so">
-          <controlPeriod>0.001</controlPeriod>
-          <robotSimType>franka_gazebo/FrankaHWSim</robotSimType>
-        </plugin>
-        <self_collide>true</self_collide>
-      </gazebo>
     </xacro:if>
     <xacro:if value="${ros2_control}">

File: robots/fer/fer.urdf.xacro (robot description, xacro)
@@ -31,4 +31,5 @@
                       kinematics="${xacro.load_yaml('$(find franka_description)/robots/$(arg arm_id)/kinematics.yaml')}"
                       dynamics="${xacro.load_yaml('$(find franka_description)/robots/$(arg arm_id)/dynamics.yaml')}"
+                      gazebo="$(arg gazebo)"
                       hand="$(arg hand)"
                       ee_id="$(arg ee_id)"

File: robots/fp3/fp3.urdf.xacro (robot description, xacro)
@@ -18,4 +18,6 @@
   <!-- Should fake sensors be used? -->
   <xacro:arg name="fake_sensor_commands" default="false" />
+  <!-- Should the robot be spawned in Gazebo?" -->
+  <xacro:arg name="gazebo" default="false" />
   <xacro:franka_robot arm_id="$(arg arm_id)"
                       joint_limits="${xacro.load_yaml('$(find franka_description)/robots/$(arg arm_id)/joint_limits.yaml')}"
@@ -23,4 +25,5 @@
                       kinematics="${xacro.load_yaml('$(find franka_description)/robots/$(arg arm_id)/kinematics.yaml')}"
                       dynamics="${xacro.load_yaml('$(find franka_description)/robots/$(arg arm_id)/dynamics.yaml')}"
+                      gazebo="$(arg gazebo)"
                       hand="$(arg hand)"
                       ee_id="$(arg ee_id)"

File: robots/fr3/fr3.urdf.xacro (robot description, xacro)
@@ -18,4 +18,6 @@
   <!-- Should fake sensors be used? -->
   <xacro:arg name="fake_sensor_commands" default="false" />
+  <!-- Should the robot be spawned in Gazebo?" -->
+  <xacro:arg name="gazebo" default="false" />
   <xacro:franka_robot arm_id="$(arg arm_id)"
                       joint_limits="${xacro.load_yaml('$(find franka_description)/robots/$(arg arm_id)/joint_limits.yaml')}"
@@ -23,4 +25,5 @@
                       kinematics="${xacro.load_yaml('$(find franka_description)/robots/$(arg arm_id)/kinematics.yaml')}"
                       dynamics="${xacro.load_yaml('$(find franka_description)/robots/$(arg arm_id)/dynamics.yaml')}"
+                      gazebo="$(arg gazebo)"
                       hand="$(arg hand)"
                       ee_id="$(arg ee_id)"

Commit message: fix: franka hand inertials fixed

File: end_effectors/common/franka_hand.xacro (robot description, xacro)
@@ -61,11 +61,9 @@
         </geometry>
       </collision>
-      <xacro:if value="${gazebo}">
-        <xacro:ee-inertials name="leftfinger" />
-      </xacro:if>
+      <xacro:ee-inertials name="leftfinger" />
     </link>
     <link name="${ee_prefix}rightfinger">
       <visual name="${ee_prefix}rightfinger_visual">
-        <origin xyz="0 0 0" rpy="0 0 ${pi}" />
+        <origin xyz="0 0 0" rpy="0 0 0" />
         <geometry>
           <mesh filename="package://${description_pkg}/meshes/robot_ee/${ee_id}/visual/finger.dae" />
@@ -74,5 +72,5 @@
       <!-- screw mount -->
       <collision>
-        <origin xyz="0 -18.5e-3 11e-3" rpy="0 0 0" />
+        <origin xyz="0 18.5e-3 11e-3" rpy="0 0 0" />
         <geometry>
           <box size="22e-3 15e-3 20e-3" />
@@ -81,5 +79,5 @@
       <!-- cartriage sledge -->
       <collision>
-        <origin xyz="0 -6.8e-3 2.2e-3" rpy="0 0 0" />
+        <origin xyz="0 6.8e-3 2.2e-3" rpy="0 0 0" />
         <geometry>
           <box size="22e-3 8.8e-3 3.8e-3" />
@@ -88,5 +86,5 @@
       <!-- diagonal finger -->
       <collision>
-        <origin xyz="0 -15.9e-3 28.35e-3" rpy="${-pi/6} 0 0" />
+        <origin xyz="0 15.9e-3 28.35e-3" rpy="${-pi/6} 0 ${pi}" />
         <geometry>
           <box size="17.5e-3 7e-3 23.5e-3" />
@@ -95,12 +93,10 @@
       <!-- rubber tip with which to grasp -->
       <collision>
-        <origin xyz="0 -7.58e-3 45.25e-3" rpy="0 0 0" />
+        <origin xyz="0 7.58e-3 45.25e-3" rpy="0 0 0" />
         <geometry>
           <box size="17.5e-3 15.2e-3 18.5e-3" />
         </geometry>
       </collision>
-      <xacro:if value="${gazebo}">
-        <xacro:ee-inertials name="rightfinger" />
-      </xacro:if>
+      <xacro:ee-inertials name="rightfinger" />
     </link>
     <joint name="${ee_prefix}finger_joint1" type="prismatic">
@@ -115,6 +111,6 @@
       <parent link="${ee_prefix}hand" />
       <child link="${ee_prefix}rightfinger" />
-      <origin xyz="0 0 0.0584" rpy="0 0 0" />
-      <axis xyz="0 -1 0" />
+      <origin xyz="0 0 0.0584" rpy="0 0 ${pi}" />
+      <axis xyz="0 1 0" />
       <limit effort="100" lower="0.0" upper="0.04" velocity="0.2" />
       <mimic joint="${ee_prefix}finger_joint1" />
