Commit message: fix: end effectors can be used for dual arm setups

File: end_effectors/cobot_pump/cobot_pump.urdf.xacro (robot description, xacro)
@@ -4,10 +4,10 @@
   <xacro:include filename="$(find franka_description)/end_effectors/common/ee_with_one_link.xacro"/>
   <xacro:include filename="$(find franka_description)/end_effectors/cobot_pump/cobot_pump_arguments.xacro"/>
-  <xacro:ee_with_one_link connected_to="$(arg connection)"
+  <xacro:ee_with_one_link connected_to="$(arg special_connection)"
                           arm_id="$(arg arm_id)"
                           ee_id="$(arg ee_id)"
                           ee_inertials="${xacro.load_yaml('$(find franka_description)/end_effectors/$(arg ee_id)/inertials.yaml')}"
-                          rpy="$(arg rpy)"
-                          xyz="$(arg xyz)"
+                          rpy_ee="$(arg rpy)"
+                          xyz_ee="$(arg xyz)"
                           tcp_xyz="$(arg tcp_xyz)"
                           tcp_rpy="$(arg tcp_rpy)"

File: end_effectors/cobot_pump/cobot_pump_arguments.xacro (robot description, xacro)
@@ -5,12 +5,12 @@
   <!-- End-effector id" -->
   <xacro:arg name="ee_id" default="cobot_pump" />
-  <!-- Where is the end-effector connected to?  -->
-  <xacro:arg name="connection" default="$(arg arm_id)_link8" />
+  <!-- Where is the end-effector connected to, if different from the robot flange?  -->
+  <xacro:arg name="special_connection" default="" />
   <!-- Should self-collision be enabled? -->
   <xacro:arg name="with_sc" default="false" />
   <!-- Position offset between ee and parent frame -->
-  <xacro:arg name="xyz" default="0 0 0" />
+  <xacro:arg name="xyz_ee" default="0 0 0" />
   <!-- Rotation offset between ee and parent frame -->
-  <xacro:arg name="rpy" default= "0 0 0" />
+  <xacro:arg name="rpy_ee" default= "0 0 0" />
   <!-- Position offset between ee frame and tcp frame -->
   <xacro:arg name="tcp_xyz" default="0 0 0.105" />

File: end_effectors/common/ee_with_one_link.xacro (robot description, xacro)
@@ -2,8 +2,8 @@
 <robot xmlns:xacro="http://www.ros.org/wiki/xacro" name="ee_with_one_link">
   <!-- safety_distance: Minimum safety distance in [m] by which the collision volumes are expanded and which is enforced during robot motions -->
-  <xacro:macro name="ee_with_one_link" params="connected_to:='' arm_id ee_id ee_inertials rpy:='0 0 0' xyz:='0 0 0' tcp_xyz:='0 0 0' tcp_rpy:='0 0 0' safety_distance:=0 gazebo:=false description_pkg:=franka_description with_sc:=false">
+  <xacro:macro name="ee_with_one_link" params="connected_to:='' arm_id arm_prefix:='' ee_id ee_inertials rpy_ee:='0 0 0' xyz_ee:='0 0 0' tcp_xyz:='0 0 0' tcp_rpy:='0 0 0' safety_distance:=0 gazebo:=false description_pkg:=franka_description with_sc:=false">
     <xacro:property name="ee_prefix" default="robot_"/>
-    <xacro:unless value="${arm_id != ''}">
-      <xacro:property name="${ee_prefix}" value="${arm_id}" />
+    <xacro:unless value="${arm_id == ''}">
+      <xacro:property name="ee_prefix" value="${arm_prefix}${arm_id}" />
     </xacro:unless>
     <xacro:unless value="${connected_to == ''}">
@@ -11,5 +11,5 @@
         <parent link="${connected_to}" />
         <child link="${ee_prefix}${ee_id}" />
-        <origin xyz="${xyz}" rpy="${rpy}" />
+        <origin xyz="${xyz_ee}" rpy="${rpy_ee}" />
       </joint>
     </xacro:unless>

File: end_effectors/common/franka_hand.xacro (robot description, xacro)
@@ -2,8 +2,8 @@
 <robot xmlns:xacro="http://www.ros.org/wiki/xacro" name="hand">
   <!-- safety_distance: Minimum safety distance in [m] by which the collision volumes are expanded and which is enforced during robot motions -->
-  <xacro:macro name="franka_hand" params="connected_to:='' arm_id ee_id ee_inertials rpy:='0 0 0' xyz:='0 0 0' tcp_xyz:='0 0 0.1034' tcp_rpy:='0 0 0' safety_distance:=0 gazebo:=false description_pkg:=franka_description with_sc:=false">
+  <xacro:macro name="franka_hand" params="connected_to:='' arm_id arm_prefix:='' ee_id ee_inertials rpy_ee:='0 0 0' xyz_ee:='0 0 0' tcp_xyz:='0 0 0.1034' tcp_rpy:='0 0 0' safety_distance:=0 gazebo:=false description_pkg:=franka_description with_sc:=false">
     <xacro:property name="ee_prefix" default="robot_"/>
-    <xacro:unless value="${arm_id != ''}">
-      <xacro:property name="${ee_prefix}" value="${arm_id}" />
+    <xacro:unless value="${arm_id == ''}">
+      <xacro:property name="ee_prefix" value="${arm_prefix}${arm_id}_" />
     </xacro:unless>
     <xacro:unless value="${connected_to == ''}">
@@ -11,5 +11,5 @@
         <parent link="${connected_to}" />
         <child link="${ee_prefix}hand" />
-        <origin xyz="${xyz}" rpy="${rpy}" />
+        <origin xyz="${xyz_ee}" rpy="${rpy_ee}" />
       </joint>
     </xacro:unless>

File: end_effectors/franka_hand/franka_hand.urdf.xacro (robot description, xacro)
@@ -4,10 +4,10 @@
   <xacro:include filename="$(find franka_description)/end_effectors/common/franka_hand.xacro"/>
   <xacro:include filename="$(find franka_description)/end_effectors/franka_hand/franka_hand_arguments.xacro"/>
-  <xacro:franka_hand connected_to="$(arg connection)"
+  <xacro:franka_hand connected_to="$(arg special_connection)"
                      arm_id="$(arg arm_id)"
                      ee_id="$(arg ee_id)_$(arg ee_color)"
                      ee_inertials="${xacro.load_yaml('$(find franka_description)/end_effectors/$(arg ee_id)/inertials.yaml')}"
-                     rpy="$(arg rpy)"
-                     xyz="$(arg xyz)"
+                     rpy_ee="$(arg rpy_ee)"
+                     xyz_ee="$(arg xyz_ee)"
                      tcp_xyz="$(arg tcp_xyz)"
                      tcp_rpy="$(arg tcp_rpy)"

File: end_effectors/franka_hand/franka_hand_arguments.xacro (robot description, xacro)
@@ -7,12 +7,12 @@
   <!-- End-effector color" -->
   <xacro:arg name="ee_color" default="white" />
-  <!-- Where is the end-effector connected to?  -->
-  <xacro:arg name="connection" default="$(arg arm_id)_link8" />
+  <!-- Where is the end-effector connected to, if different from the robot flange?  -->
+  <xacro:arg name="special_connection" default="" />
   <!-- Should self-collision be enabled? -->
   <xacro:arg name="with_sc" default="false" />
   <!-- Position offset between ee and parent frame -->
-  <xacro:arg name="xyz" default="0 0 0" />
+  <xacro:arg name="xyz_ee" default="0 0 0" />
   <!-- Rotation offset between ee and parent frame -->
-  <xacro:arg name="rpy" default= "0 0 ${-pi/4}" />
+  <xacro:arg name="rpy_ee" default= "0 0 ${-pi/4}" />
   <!-- Position offset between ee frame and tcp frame -->
   <xacro:arg name="tcp_xyz" default="0 0 0.1034" />

File: robots/common/franka_robot.xacro (robot description, xacro)
@@ -49,11 +49,14 @@
         <xacro:property name="ee_color" value="white" />
       </xacro:if>
+      <xacro:property name="special_connection" value="$(arg special_connection)" />
+      <xacro:property name="connection" value="${special_connection if special_connection != '' else arm_id + '_link8'}" />
       <xacro:franka_hand
-        connected_to="$(arg connection)"
+        connected_to="${arm_prefix}${connection}"
         arm_id="${arm_id}"
+        arm_prefix="${arm_prefix}"
         ee_id="${ee_id}_${ee_color}"
         ee_inertials="${xacro.load_yaml('$(find franka_description)/end_effectors/$(arg ee_id)/inertials.yaml')}"
-        rpy="$(arg rpy)"
-        xyz="$(arg xyz)"
+        rpy_ee="$(arg rpy_ee)"
+        xyz_ee="$(arg xyz_ee)"
         tcp_xyz="$(arg tcp_xyz)"
         tcp_rpy="$(arg tcp_rpy)"
@@ -68,11 +71,14 @@
       <xacro:include filename="$(find franka_description)/end_effectors/common/utils.xacro" />
       <xacro:include filename="$(find franka_description)/end_effectors/$(arg ee_id)/$(arg ee_id)_arguments.xacro" />
+      <xacro:property name="special_connection" value="$(arg special_connection)" />
+      <xacro:property name="connection" value="${special_connection if special_connection == '' else arm_id + '_link8'}" />
       <xacro:ee_with_one_link
-        connected_to="$(arg connection)"
+        connected_to="${arm_prefix}${connection}"
         arm_id="${arm_id}"
+        arm_prefix="${arm_prefix}"
         ee_id="${ee_id}"
         ee_inertials="${xacro.load_yaml('$(find franka_description)/end_effectors/$(arg ee_id)/inertials.yaml')}"
-        rpy="$(arg rpy)"
-        xyz="$(arg xyz)"
+        rpy_ee="$(arg rpy_ee)"
+        xyz_ee="$(arg xyz_ee)"
         tcp_xyz="$(arg tcp_xyz)"
         tcp_rpy="$(arg tcp_rpy)"

File: robots/multi_arm/multi_arm.urdf.xacro (robot description, xacro)
@@ -12,8 +12,8 @@
   <xacro:arg name="number_of_robots" default = "2"/>
   <!-- Define arguments -->
-  <xacro:arg name="xyz" default="['0.5 0.5 0','0 0 0']" />
+  <xacro:arg name="xyz" default="['0 0.1 0','0 -0.1 0']" />
   <xacro:property name="xyz_list" value="${$(arg xyz)}" />
   <!-- Define arguments -->
-  <xacro:arg name="rpy" default="['0 0 0','0 0 0']" />
+  <xacro:arg name="rpy" default="['-0.7 0 0','0.7 0 0']" />
   <xacro:property name="rpy_list" value="${$(arg rpy)}" />
   <!-- Don't print a prefix for joints, visuals, and links? -->

Commit message: fix: creating urdf with cobot pump

File: end_effectors/cobot_pump/cobot_pump.urdf.xacro (robot description, xacro)
@@ -8,6 +8,6 @@
                           ee_id="$(arg ee_id)"
                           ee_inertials="${xacro.load_yaml('$(find franka_description)/end_effectors/$(arg ee_id)/inertials.yaml')}"
-                          rpy_ee="$(arg rpy)"
-                          xyz_ee="$(arg xyz)"
+                          rpy_ee="$(arg rpy_ee)"
+                          xyz_ee="$(arg xyz_ee)"
                           tcp_xyz="$(arg tcp_xyz)"
                           tcp_rpy="$(arg tcp_rpy)"

File: end_effectors/common/ee_with_one_link.xacro (robot description, xacro)
@@ -5,5 +5,5 @@
     <xacro:property name="ee_prefix" default="robot_"/>
     <xacro:unless value="${arm_id == ''}">
-      <xacro:property name="ee_prefix" value="${arm_prefix}${arm_id}" />
+      <xacro:property name="ee_prefix" value="${arm_prefix}${arm_id}_" />
     </xacro:unless>
     <xacro:unless value="${connected_to == ''}">
